Commit message: Choose one URDF model from shadowhands package and visualize.
  - Modify the original URDF to place both hands in a better location.

File: sr_description/robots/bimanual_shadowhand_motor.urdf.xacro (robot description, xacro)
@@ -8,5 +8,6 @@
     <parent link="world" />
     <child link="rh_forearm" />
-    <origin xyz="0.0 0.0 0.0" rpy="0.0 0.0 0.0" />
+    <!--origin xyz="0.0 0.0 0.0" rpy="0.0 0.0 0.0" /-->
+    <origin xyz="-0.2 0.0 0.0" rpy="0.0 0.0 0.0" /> <!-- Modified by LYW, 2020-11-04 -->
   </joint>
   <xacro:shadowhand muscletrans="false" muscle="false" bio="false" bt_sp="false"
