Commit message: Test using PositionJointInterface, but the PID is not easy to tune... So give up and turn to MoveIt.

File: sr_description/hand/xacro/finger/distal/distal.transmission.xacro (robot description, xacro)
@@ -28,9 +28,9 @@
             <actuator name="${prefix}${joint_prefix}J1">
                 <mechanicalReduction>1</mechanicalReduction>
-                <hardwareInterface>hardware_interface/EffortJointInterface</hardwareInterface>
+                <hardwareInterface>hardware_interface/PositionJointInterface</hardwareInterface>
             </actuator>
             <joint name="${prefix}${joint_prefix}J1">
                 <!--hardwareInterface>hardwareInterface/EffortJointInterface</hardwareInterface-->
-                <hardwareInterface>hardware_interface/EffortJointInterface</hardwareInterface>
+                <hardwareInterface>hardware_interface/PositionJointInterface</hardwareInterface>
             </joint>
         </transmission>

File: sr_description/hand/xacro/finger/knuckle/knuckle.transmission.xacro (robot description, xacro)
@@ -28,9 +28,9 @@
                 <actuator name="${prefix}${joint_prefix}J4">
                     <mechanicalReduction>1</mechanicalReduction>
-                    <hardwareInterface>hardware_interface/EffortJointInterface</hardwareInterface>
+                    <hardwareInterface>hardware_interface/PositionJointInterface</hardwareInterface>
                 </actuator>
                 <joint name="${prefix}${joint_prefix}J4">
                     <!--hardwareInterface>EffortJointInterface</hardwareInterface-->
-                    <hardwareInterface>hardware_interface/EffortJointInterface</hardwareInterface>
+                    <hardwareInterface>hardware_interface/PositionJointInterface</hardwareInterface>
                 </joint>
             </transmission>

File: sr_description/hand/xacro/finger/lfmetacarpal/lfmetacarpal.transmission.xacro (robot description, xacro)
@@ -26,9 +26,9 @@
                 <actuator name="${prefix}LFJ5">
                     <mechanicalReduction>1</mechanicalReduction>
-                    <hardwareInterface>hardware_interface/EffortJointInterface</hardwareInterface>
+                    <hardwareInterface>hardware_interface/PositionJointInterface</hardwareInterface>
                 </actuator>
                 <joint name="${prefix}LFJ5">
                     <!--hardwareInterface>EffortJointInterface</hardwareInterface-->
-                    <hardwareInterface>hardware_interface/EffortJointInterface</hardwareInterface>
+                    <hardwareInterface>hardware_interface/PositionJointInterface</hardwareInterface>
                 </joint>
             </transmission>

File: sr_description/hand/xacro/finger/middle/middle.transmission.xacro (robot description, xacro)
@@ -34,11 +34,24 @@
                 <actuator name="${prefix}${joint_prefix}J0">
                     <mechanicalReduction>1</mechanicalReduction>
-                    <hardwareInterface>hardware_interface/EffortJointInterface</hardwareInterface>
+                    <hardwareInterface>hardware_interface/PositionJointInterface</hardwareInterface>
                 </actuator>
                 <joint name="${prefix}${joint_prefix}J1">
                     <!--hardwareInterface>EffortJointInterface</hardwareInterface-->
-                    <hardwareInterface>hardware_interface/EffortJointInterface</hardwareInterface>
+                    <hardwareInterface>hardware_interface/PositionJointInterface</hardwareInterface>
                 </joint>
-                <secondJoint name="${prefix}${joint_prefix}J2"/>
+                <!-- <secondJoint name="${prefix}${joint_prefix}J2"/> -->
+            </transmission>
+            <!-- Added by LYW, 2020-11-05: Separate the coupled joint -->
+            <transmission name="${prefix}${link_prefix}middle_transmission2">
+                <!--type>sr_mechanism_model/J0Transmission</type-->
+                <type>transmission_interface/SimpleTransmission</type>
+                <actuator name="${prefix}${joint_prefix}J1">
+                    <mechanicalReduction>1</mechanicalReduction>
+                    <hardwareInterface>hardware_interface/PositionJointInterface</hardwareInterface>
+                </actuator>
+                <joint name="${prefix}${joint_prefix}J2">
+                    <!--hardwareInterface>EffortJointInterface</hardwareInterface-->
+                    <hardwareInterface>hardware_interface/PositionJointInterface</hardwareInterface>
+                </joint>
             </transmission>
         </xacro:unless>

File: sr_description/hand/xacro/finger/proximal/proximal.transmission.xacro (robot description, xacro)
@@ -28,9 +28,9 @@
                 <actuator name="${prefix}${joint_prefix}J3">
                     <mechanicalReduction>1</mechanicalReduction>
-                    <hardwareInterface>hardware_interface/EffortJointInterface</hardwareInterface>
+                    <hardwareInterface>hardware_interface/PositionJointInterface</hardwareInterface>
                 </actuator>
                 <joint name="${prefix}${joint_prefix}J3">
                     <!--hardwareInterface>EffortJointInterface</hardwareInterface-->
-                    <hardwareInterface>hardware_interface/EffortJointInterface</hardwareInterface>
+                    <hardwareInterface>hardware_interface/PositionJointInterface</hardwareInterface>
                 </joint>
             </transmission>

File: sr_description/hand/xacro/palm/palm.transmission.xacro (robot description, xacro)
@@ -26,9 +26,9 @@
                 <actuator name="${prefix}WRJ1">
                     <mechanicalReduction>1</mechanicalReduction>
-                    <hardwareInterface>hardware_interface/EffortJointInterface</hardwareInterface>
+                    <hardwareInterface>hardware_interface/PositionJointInterface</hardwareInterface>
                 </actuator>
                 <joint name="${prefix}WRJ1">
                     <!--hardwareInterface>EffortJointInterface</hardwareInterface-->
-                    <hardwareInterface>hardware_interface/EffortJointInterface</hardwareInterface>
+                    <hardwareInterface>hardware_interface/PositionJointInterface</hardwareInterface>
                 </joint>
             </transmission>

File: sr_description/hand/xacro/thumb/thbase.transmission.xacro (robot description, xacro)
@@ -26,9 +26,9 @@
                 <actuator name="${prefix}THJ5">
                     <mechanicalReduction>1</mechanicalReduction>
-                    <hardwareInterface>hardware_interface/EffortJointInterface</hardwareInterface>
+                    <hardwareInterface>hardware_interface/PositionJointInterface</hardwareInterface>
                 </actuator>
                 <joint name="${prefix}THJ5">
                     <!--hardwareInterface>EffortJointInterface</hardwareInterface-->
-                    <hardwareInterface>hardware_interface/EffortJointInterface</hardwareInterface>
+                    <hardwareInterface>hardware_interface/PositionJointInterface</hardwareInterface>
                 </joint>
             </transmission>

File: sr_description/hand/xacro/thumb/thdistal.transmission.xacro (robot description, xacro)
@@ -26,9 +26,9 @@
                 <actuator name="${prefix}THJ1">
                     <mechanicalReduction>1</mechanicalReduction>
-                    <hardwareInterface>hardware_interface/EffortJointInterface</hardwareInterface>
+                    <hardwareInterface>hardware_interface/PositionJointInterface</hardwareInterface>
                 </actuator>
                 <joint name="${prefix}THJ1">
                     <!--hardwareInterface>EffortJointInterface</hardwareInterface-->
-                    <hardwareInterface>hardware_interface/EffortJointInterface</hardwareInterface>
+                    <hardwareInterface>hardware_interface/PositionJointInterface</hardwareInterface>
                 </joint>
             </transmission>

File: sr_description/hand/xacro/thumb/thhub.transmission.xacro (robot description, xacro)
@@ -26,9 +26,9 @@
                 <actuator name="${prefix}THJ3">
                     <mechanicalReduction>1</mechanicalReduction>
-                    <hardwareInterface>hardware_interface/EffortJointInterface</hardwareInterface>
+                    <hardwareInterface>hardware_interface/PositionJointInterface</hardwareInterface>
                 </actuator>
                 <joint name="${prefix}THJ3">
                     <!--hardwareInterface>EffortJointInterface</hardwareInterface-->
-                    <hardwareInterface>hardware_interface/EffortJointInterface</hardwareInterface>
+                    <hardwareInterface>hardware_interface/PositionJointInterface</hardwareInterface>
                 </joint>
             </transmission>

File: sr_description/hand/xacro/thumb/thmiddle.transmission.xacro (robot description, xacro)
@@ -26,9 +26,9 @@
                 <actuator name="${prefix}THJ2">
                     <mechanicalReduction>1</mechanicalReduction>
-                    <hardwareInterface>hardware_interface/EffortJointInterface</hardwareInterface>
+                    <hardwareInterface>hardware_interface/PositionJointInterface</hardwareInterface>
                 </actuator>
                 <joint name="${prefix}THJ2">
                     <!--hardwareInterface>EffortJointInterface</hardwareInterface-->
-                    <hardwareInterface>hardware_interface/EffortJointInterface</hardwareInterface>
+                    <hardwareInterface>hardware_interface/PositionJointInterface</hardwareInterface>
                 </joint>
             </transmission>

File: sr_description/hand/xacro/thumb/thproximal.transmission.xacro (robot description, xacro)
@@ -26,9 +26,9 @@
                 <actuator name="${prefix}THJ4">
                     <mechanicalReduction>1</mechanicalReduction>
-                    <hardwareInterface>hardware_interface/EffortJointInterface</hardwareInterface>
+                    <hardwareInterface>hardware_interface/PositionJointInterface</hardwareInterface>
                 </actuator>
                 <joint name="${prefix}THJ4">
                     <!--hardwareInterface>EffortJointInterface</hardwareInterface-->
-                    <hardwareInterface>hardware_interface/EffortJointInterface</hardwareInterface>
+                    <hardwareInterface>hardware_interface/PositionJointInterface</hardwareInterface>
                 </joint>
             </transmission>

File: sr_description/hand/xacro/wrist/wrist.transmission.xacro (robot description, xacro)
@@ -26,9 +26,9 @@
                 <actuator name="${prefix}WRJ2">
                     <mechanicalReduction>1</mechanicalReduction>
-                    <hardwareInterface>hardware_interface/EffortJointInterface</hardwareInterface>
+                    <hardwareInterface>hardware_interface/PositionJointInterface</hardwareInterface>
                 </actuator>
                 <joint name="${prefix}WRJ2">
                     <!--hardwareInterface>EffortJointInterface</hardwareInterface-->
-                    <hardwareInterface>hardware_interface/EffortJointInterface</hardwareInterface>
+                    <hardwareInterface>hardware_interface/PositionJointInterface</hardwareInterface>
                 </joint>
             </transmission>
